File: hardware/ind_heater/ind_heater.sch (KiCad schematic (older format))
At the start: 16 parts, among them J1 DG126-5.0-02P, J2 Conn_01x01_Male, J3 Conn_01x01_Male, J4 Conn_01x01_Male, Q1 IRFZ46N, Q2 IRFZ46N

Commit message: тестовая плата собрана, но не проверена
Parts:
- J1: symbol Connector_Degson:DG126-5.0-02P -> ind_heater-rescue:DG126-5.0-02P-Connector_Degson
- Q1, Q2: symbol Transistor_FET:IRFZ46N -> ind_heater-rescue:IRFZ46N-Transistor_FET
Changed lines of the file:
@@
 $EndDescr
 $Comp
-L Transistor_FET:IRFZ46N Q1
+L ind_heater-rescue:IRFZ46N-Transistor_FET Q1
 U 1 1 5EB19214
 P 5450 4000
@@
 $EndComp
 $Comp
-L Connector_Degson:DG126-5.0-02P J1
+L ind_heater-rescue:DG126-5.0-02P-Connector_Degson J1
 U 1 1 5EAE9A9B
 P 2900 3950
@@
 $EndComp
 $Comp
-L Transistor_FET:IRFZ46N Q2
+L ind_heater-rescue:IRFZ46N-Transistor_FET Q2
 U 1 1 5EAF3120
 P 5450 4600
